Commit message: add imu node

File: pinky_description/urdf/pinky.urdf.xacro (robot description, xacro)
@@ -216,4 +216,10 @@
             <origin xyz="0.0295 -0.02 -0.015" rpy="0 0 0"/>
         </joint>
+        <link name="imu_link"/>
+        <joint name="imu_fixed_joint" type="fixed">
+            <parent link="base_link"/>
+            <child link="imu_link"/>
+            <origin xyz="-0.044 0 0.0525" rpy="0 0 0"/>
+        </joint>
         <xacro:insert_ros2_control name="pinky"/>
     </xacro:macro>

Commit message: Add front_camera and argument for adjust camera tilt angle

File: pinky_description/urdf/pinky.urdf.xacro (robot description, xacro)
@@ -1,5 +1,5 @@
 <?xml version="1.0"?>
 <robot xmlns:xacro="http://www.ros.org/wiki/xacro">
-    <xacro:macro name="insert_robot" params="namespace">
+    <xacro:macro name="insert_robot" params="namespace front_camera_tilt_deg">
         <xacro:include filename="$(find pinky_description)/urdf/common/insert_inertia.urdf.xacro"/>
         <xacro:include filename="$(find pinky_description)/urdf/pinky_ros2_control.urdf.xacro"/>
@@ -186,9 +186,33 @@
             <origin xyz="0 0 0.030" rpy="0 0 0"/>
         </joint>
+        <link name="front_camera_mount">
+            <visual>
+                <origin xyz="0 0 0" rpy="0 0 0"/>
+                <geometry>
+                    <mesh filename="package://pinky_description/meshes/visual/front_camera_mount.dae" scale="1 1 1"/>
+                </geometry>
+            </visual>
+            <collision>
+                <origin xyz="0 0 0" rpy="0 0 0"/>
+                <geometry>
+                    <mesh filename="package://pinky_description/meshes/collision/front_camera_mount.stl" scale="1 1 1"/>
+                </geometry>
+            </collision>
+            <inertial>
+                <origin xyz="-0.06425 0 0.078" rpy="0 0 0"/>
+                <mass value="0.01"/>
+                <xacro:box_inertia m="0.01" x="0.0165" y="0.058" z="0.018"/>
+            </inertial>
+        </link>
+        <joint name="front_camera_mount_fixed_joint" type="fixed">
+            <parent link="base_link"/>
+            <child link="front_camera_mount"/>
+            <origin xyz="0.020 0 0.0495" rpy="0 ${front_camera_tilt_deg/180*pi} 0"/>
+        </joint>
         <link name="front_camera_link"/>
         <joint name="front_camera_fixed_joint" type="fixed">
-            <parent link="base_link"/>
+            <parent link="front_camera_mount"/>
             <child link="front_camera_link"/>
-            <origin xyz="0.032 0 0.0345" rpy="0 0 0"/>
+            <origin xyz="0.015 0 -0.0121" rpy="0 0 0"/>
         </joint>
         <link name="ultrasonic_link"/>

File: pinky_description/urdf/robot.urdf.xacro (robot description, xacro)
@@ -2,5 +2,6 @@
 <robot xmlns:xacro="http://ros.org/wiki/xacro" name="pinky">
     <xacro:include filename="$(find pinky_description)/urdf/pinky.urdf.xacro"/>
+    <xacro:arg name="front_camera_tilt_deg" default="0.0"/>
     <xacro:arg name="namespace" default=""/>
-    <xacro:insert_robot namespace="$(arg namespace)"/>
+    <xacro:insert_robot namespace="$(arg namespace)" front_camera_tilt_deg="$(arg front_camera_tilt_deg)"/>
 </robot>

Commit message: bug fixed

File: pinky_description/urdf/pinky.urdf.xacro (robot description, xacro)
@@ -200,7 +200,7 @@
             </collision>
             <inertial>
-                <origin xyz="-0.06425 0 0.078" rpy="0 0 0"/>
+                <origin xyz="0.01 0 -0.0121" rpy="0 0 0"/>
                 <mass value="0.01"/>
-                <xacro:box_inertia m="0.01" x="0.0165" y="0.058" z="0.018"/>
+                <xacro:box_inertia m="0.01" x="0.0165" y="0.045" z="0.030"/>
             </inertial>
         </link>

Commit message: Add support for gz_sim

File: pinky_description/urdf/pinky.urdf.xacro (robot description, xacro)
@@ -1,5 +1,5 @@
 <?xml version="1.0"?>
 <robot xmlns:xacro="http://www.ros.org/wiki/xacro">
-    <xacro:macro name="insert_robot" params="namespace front_camera_tilt_deg">
+    <xacro:macro name="insert_robot" params="namespace is_sim:=false sim_type:=gz_sim cam_tilt_deg">
         <xacro:include filename="$(find pinky_description)/urdf/common/insert_inertia.urdf.xacro"/>
         <xacro:include filename="$(find pinky_description)/urdf/pinky_ros2_control.urdf.xacro"/>
@@ -208,5 +208,5 @@
             <parent link="base_link"/>
             <child link="front_camera_mount"/>
-            <origin xyz="0.020 0 0.0495" rpy="0 ${front_camera_tilt_deg/180*pi} 0"/>
+            <origin xyz="0.020 0 0.0495" rpy="0 ${cam_tilt_deg/180*pi} 0"/>
         </joint>
         <link name="front_camera_link"/>
@@ -246,5 +246,11 @@
             <origin xyz="-0.044 0 0.0525" rpy="0 0 0"/>
         </joint>
-        <xacro:insert_ros2_control name="pinky"/>
+        <xacro:if value="${is_sim}">
+            <xacro:if value="${sim_type == 'gz_sim'}">
+                <xacro:include filename="$(find pinky_description)/urdf/pinky_gz.urdf.xacro"/>
+                <xacro:insert_gz_sim namespace="${namespace}"/>
+            </xacro:if>
+        </xacro:if>
+        <xacro:insert_ros2_control name="pinky" is_sim="${is_sim}" sim_type="${sim_type}"/>
     </xacro:macro>
 </robot>

File: pinky_description/urdf/pinky_ros2_control.urdf.xacro (robot description, xacro)
@@ -1,12 +1,29 @@
 <?xml version="1.0"?>
 <robot xmlns:xacro="http://www.ros.org/wiki/xacro">
-    <xacro:macro name="insert_ros2_control" params="name">
+    <xacro:macro name="insert_ros2_control" params="name is_sim sim_type">
         <ros2_control name="${name}_system" type="system">
-            <hardware>
-                <plugin>pinky_hardware_interface/PinkySystemHardwareInterface</plugin>
-                <param name="interface_name">/dev/ttyAMA4</param>
-                <param name="profile_acceleration">500</param>
-                <param name="profile_velocity">1620</param>
-            </hardware>
+            <xacro:if value="${is_sim}">
+                <xacro:if value="${sim_type == 'gz_sim'}">
+                    <hardware>
+                        <plugin>gz_ros2_control/GazeboSimSystem</plugin>
+                    </hardware>
+                </xacro:if>
+                <xacro:if value="${sim_type == 'isaacsim'}">
+                    <hardware>
+                        <plugin>topic_based_ros2_control/TopicBasedSystem</plugin>
+                        <param name="joint_commands_topic">isaac_pinky_joint_commands</param>
+                        <param name="joint_states_topic">isaac_pinky_joint_states</param>
+                        <param name="sum_wrapped_joint_states">true</param>
+                    </hardware>
+                </xacro:if>
+            </xacro:if>
+            <xacro:unless value="${is_sim}">
+                <hardware>
+                    <plugin>pinky_hardware_interface/PinkySystemHardwareInterface</plugin>
+                    <param name="interface_name">/dev/ttyAMA4</param>
+                    <param name="profile_acceleration">500</param>
+                    <param name="profile_velocity">1620</param>
+                </hardware>
+            </xacro:unless>
             <joint name="l_wheel_joint">
                 <command_interface name="velocity">
@@ -27,18 +44,20 @@
                 <state_interface name="effort" />
             </joint>
-            <gpio name="gpio">
-                <command_interface name="enable_torque" />
-                <command_interface name="set_led" />
-                <state_interface name="l_motor_enabled" />
-                <state_interface name="l_motor_hw_error_status" />
-                <state_interface name="l_motor_present_voltage" />
-                <state_interface name="l_motor_present_temp" />
-                <state_interface name="l_motor_led"/>
-                <state_interface name="r_motor_enabled" />
-                <state_interface name="r_motor_hw_error_status" />
-                <state_interface name="r_motor_present_voltage" />
-                <state_interface name="r_motor_present_temp" />
-                <state_interface name="r_motor_led"/>
-            </gpio>
+            <xacro:unless value="${is_sim}">
+                <gpio name="gpio">
+                    <command_interface name="enable_torque" />
+                    <command_interface name="set_led" />
+                    <state_interface name="l_motor_enabled" />
+                    <state_interface name="l_motor_hw_error_status" />
+                    <state_interface name="l_motor_present_voltage" />
+                    <state_interface name="l_motor_present_temp" />
+                    <state_interface name="l_motor_led"/>
+                    <state_interface name="r_motor_enabled" />
+                    <state_interface name="r_motor_hw_error_status" />
+                    <state_interface name="r_motor_present_voltage" />
+                    <state_interface name="r_motor_present_temp" />
+                    <state_interface name="r_motor_led"/>
+                </gpio>
+            </xacro:unless>
         </ros2_control>
     </xacro:macro>

File: pinky_description/urdf/robot.urdf.xacro (robot description, xacro)
@@ -2,6 +2,12 @@
 <robot xmlns:xacro="http://ros.org/wiki/xacro" name="pinky">
     <xacro:include filename="$(find pinky_description)/urdf/pinky.urdf.xacro"/>
-    <xacro:arg name="front_camera_tilt_deg" default="0.0"/>
+    <xacro:arg name="cam_tilt_deg" default="0.0"/>
+    <xacro:arg name="is_sim" default="true"/>
+    <xacro:arg name="sim_type" default="gz_sim"/>   <!-- gz_sim / isaacsim -->
     <xacro:arg name="namespace" default=""/>
-    <xacro:insert_robot namespace="$(arg namespace)" front_camera_tilt_deg="$(arg front_camera_tilt_deg)"/>
+    <xacro:insert_robot namespace="$(arg namespace)"
+                        is_sim="$(arg is_sim)"
+                        sim_type="$(arg sim_type)"
+                        cam_tilt_deg="$(arg cam_tilt_deg)"
+    />
 </robot>

Commit message: bug fixed

File: pinky_description/urdf/pinky.urdf.xacro (robot description, xacro)
@@ -178,5 +178,5 @@
             <parent link="base_link"/>
             <child link="rplidar_mount"/>
-            <origin xyz="-0.017 0 0.067" rpy="0 0 0"/>
+            <origin xyz="-0.017 0 0.067" rpy="0 0 ${pi}"/>
         </joint>
         <link name="rplidar_link"/>

Commit message: feat: update pinky pkg (thanks to @byeongkyu)

File: pinky_description/urdf/pinky.urdf.xacro (robot description, xacro)
@@ -1,5 +1,5 @@
 <?xml version="1.0"?>
 <robot xmlns:xacro="http://www.ros.org/wiki/xacro">
-    <xacro:macro name="insert_robot" params="namespace is_sim:=false sim_type:=gz_sim cam_tilt_deg">
+    <xacro:macro name="insert_robot" params="namespace is_sim:=false sim_type:=gz_sim cam_tilt_deg screen_tilt_deg">
         <xacro:include filename="$(find pinky_description)/urdf/common/insert_inertia.urdf.xacro"/>
         <xacro:include filename="$(find pinky_description)/urdf/pinky_ros2_control.urdf.xacro"/>
@@ -117,5 +117,5 @@
                 <origin xyz="0 0 0" rpy="0 0 0"/>
                 <geometry>
-                    <sphere radius="0.00625"/>
+                    <sphere radius="0.0065"/>
                 </geometry>
             </collision>
@@ -123,5 +123,5 @@
                 <origin xyz="0 0 0" rpy="0 0 0"/>
                 <mass value="0.05"/>
-                <xacro:sphere_inertia m="0.05" r="0.00625"/>
+                <xacro:sphere_inertia m="0.05" r="0.0065"/>
             </inertial>
         </link>
@@ -178,5 +178,5 @@
             <parent link="base_link"/>
             <child link="rplidar_mount"/>
-            <origin xyz="-0.017 0 0.067" rpy="0 0 ${pi}"/>
+            <origin xyz="-0.017 0 0.067" rpy="0 0 0"/>
         </joint>
         <link name="rplidar_link"/>
@@ -184,5 +184,5 @@
             <parent link="rplidar_mount"/>
             <child link="rplidar_link"/>
-            <origin xyz="0 0 0.030" rpy="0 0 0"/>
+            <origin xyz="0 0 0.030" rpy="0 0 ${pi}"/>
         </joint>
         <link name="front_camera_mount">
@@ -190,11 +190,11 @@
                 <origin xyz="0 0 0" rpy="0 0 0"/>
                 <geometry>
-                    <mesh filename="package://pinky_description/meshes/visual/front_camera_mount.dae" scale="1 1 1"/>
-                </geometry>
-            </visual>
-            <collision>
-                <origin xyz="0 0 0" rpy="0 0 0"/>
-                <geometry>
-                    <mesh filename="package://pinky_description/meshes/collision/front_camera_mount.stl" scale="1 1 1"/>
+                    <mesh filename="package://pinky_description/meshes/visual/camera_assy.dae" scale="1 1 1"/>
+                </geometry>
+            </visual>
+            <collision>
+                <origin xyz="0 0 0" rpy="0 0 0"/>
+                <geometry>
+                    <mesh filename="package://pinky_description/meshes/collision/camera_assy.stl" scale="1 1 1"/>
                 </geometry>
             </collision>
@@ -215,4 +215,28 @@
             <child link="front_camera_link"/>
             <origin xyz="0.015 0 -0.0121" rpy="0 0 0"/>
+        </joint>
+        <link name="screen_mount">
+            <visual>
+                <origin xyz="0 0 0" rpy="0 0 0"/>
+                <geometry>
+                    <mesh filename="package://pinky_description/meshes/visual/screen_assy.dae" scale="1 1 1"/>
+                </geometry>
+            </visual>
+            <collision>
+                <origin xyz="0 0 0" rpy="0 0 0"/>
+                <geometry>
+                    <mesh filename="package://pinky_description/meshes/collision/screen_assy.stl" scale="1 1 1"/>
+                </geometry>
+            </collision>
+            <inertial>
+                <origin xyz="0.01 0 -0.004" rpy="0 0 0"/>
+                <mass value="0.01"/>
+                <xacro:box_inertia m="0.01" x="0.012" y="0.071" z="0.041"/>
+            </inertial>
+        </link>
+        <joint name="screen_mount_fixed_joint" type="fixed">
+            <parent link="base_link"/>
+            <child link="screen_mount"/>
+            <origin xyz="0.0165 0 0.071" rpy="0 ${screen_tilt_deg/180*pi} 0"/>
         </joint>
         <link name="ultrasonic_link"/>

File: pinky_description/urdf/pinky_ros2_control.urdf.xacro (robot description, xacro)
@@ -11,7 +11,7 @@
                 <xacro:if value="${sim_type == 'isaacsim'}">
                     <hardware>
-                        <plugin>topic_based_ros2_control/TopicBasedSystem</plugin>
-                        <param name="joint_commands_topic">isaac_pinky_joint_commands</param>
-                        <param name="joint_states_topic">isaac_pinky_joint_states</param>
+                        <plugin>joint_state_topic_hardware_interface/JointStateTopicSystem</plugin>
+                        <param name="joint_commands_topic">/isaacsim_pinky_joint_command</param>
+                        <param name="joint_states_topic">/isaacsim_pinky_joint_states</param>
                         <param name="sum_wrapped_joint_states">true</param>
                     </hardware>

File: pinky_description/urdf/robot.urdf.xacro (robot description, xacro)
@@ -5,5 +5,10 @@
     <xacro:arg name="is_sim" default="false"/>
     <xacro:arg name="sim_type" default="gz_sim"/>
-    <xacro:arg name="cam_tilt_deg" default="0"/>
-    <xacro:insert_robot namespace="$(arg namespace)" is_sim="$(arg is_sim)" sim_type="$(arg sim_type)" cam_tilt_deg="$(arg cam_tilt_deg)"/>
+    <xacro:arg name="cam_tilt_deg" default="8"/>
+    <xacro:arg name="screen_tilt_deg" default="-25"/>
+    <xacro:insert_robot namespace="$(arg namespace)"
+                        is_sim="$(arg is_sim)"
+                        sim_type="$(arg sim_type)"
+                        cam_tilt_deg="$(arg cam_tilt_deg)"
+                        screen_tilt_deg="$(arg screen_tilt_deg)"/>
 </robot>
